File: CHIRIMENBasicShield/CHIRIMENBasicShield.sch (EAGLE design)
At the start: 17 parts, among them J1 4P-2.0, J10 4P-2.0-90D, J2 4P-2.0, J3 4P-2.0, J4 4P-2.0, J5 4P-2.0, J6 4P-2.0, J7 4P-2.0, J8 4P-2.0, J9 4P-2.0-90D

Commit message: issues #45,46
Connections:
- removed net N$12: CN1.18, J7.3, J8.3, J9.3
- removed net N$2 (its old number): ADT4710.1, CN2.18, J10.3, J3.3, J4.3, SRF02.1
- removed net N$8: CN1.17, J1.3, J5.3, J6.3
- new net 3V3: CN1.17, J1.3, J2.3, J5.3, J6.3
- new net 5V: ADT4710.1, CN1.18, J10.3, J3.3, J4.3, J7.3, J8.3, J9.3, SRF02.1
Other:
- moved on the sheet: GND, J1, J10, J2, J3, J4, J5, J6, J7, J8, J9
